File: KeyboardRev1.kicad_pcb (KiCad board)
At the start: 2 copper layers, 157 parts, among them J1 ISP, SW1 RESET, SW10 8, SW11 9, SW12 0, SW13 -_, SW14 =+, SW15 BSPC, SW16 PGUP, SW17 Tab, SW18 Q, SW19 W, SW2 GRV, SW20 E, SW21 R, SW22 T, SW23 Y, SW24 U, SW25 I, SW26 O, SW27 P, SW28 [{, SW29 ]}, SW3 1, SW30 \|, SW31 PGDN, SW32 CAPS, SW33 A, SW34 S, SW35 D, SW36 F, SW37 G, SW38 H, SW39 J, SW4 2, SW40 K, SW41 L, SW42 ;:, SW43 '", SW45 ENTER, SW46 DEL, SW47 LSHIFT, SW48 Z, SW49 X, SW5 3, SW50 C, SW51 V, SW52 B, SW53 N, SW54 M, SW55 ,<, SW56 .>, SW57 /?, SW59 RSHIFT, SW6 4, SW60 UP, SW61 END, SW62 LCTL, SW63 WIN, SW64 LALT, SW68 SPC, SW7 5, SW72 FN, SW73 RCTL, SW74 LEFT, SW75 DOWN, SW76 RIGHT, SW77 RALT, SW8 6, SW9 7, U1 MCU, U2 PRTR5V0U2X, Y1 16MHz

Commit message: Updated PCB, Currently finishing cooper traces
Parts:
- moved USB1 325.5 mm to (208.3, 28.0), turned to 0 degrees
- moved R6 310.0 mm to (204.0, 39.7)
- moved U2 306.3 mm to (207.8, 46.0)
- moved R5 305.3 mm to (210.3, 39.7), turned to 0 degrees
- moved F1 305.1 mm to (202.7, 46.8), turned to -90 degrees
- moved C8 254.3 mm to (202.5, 108.0)
- moved C5 242.5 mm to (200.8, 112.8), turned to -90 degrees
- moved R4 242.2 mm to (205.7, 105.5), turned to -90 degrees
- moved R3 238.7 mm to (207.9, 105.5), turned to -90 degrees
- moved C6 238.0 mm to (200.8, 120.7), turned to 90 degrees
- moved C7 232.6 mm to (213.5, 123.9), turned to 0 degrees
- moved C1 232.5 mm to (212.3, 106.5), turned to 0 degrees
- moved C4 231.9 mm to (218.3, 113.6), turned to -90 degrees
- moved U1 224.5 mm to (209.5, 116.0), turned to -90 degrees
- moved C2 219.9 mm to (230.2, 115.9), turned to -90 degrees
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Connections:
- net Net-(U2-IO1) renamed DP
- net Net-(U2-IO2) renamed DN
- SW68 pad 2: col6 -> col5
Routing:
- net row0: track 0.00 -> 285.2 mm, vias 0 -> 2
- net row4: track 0.00 -> 279.9 mm, vias 0 -> 2
- net row1: track 0.00 -> 275.9 mm, vias 0 -> 2
- net row2: track 0.00 -> 267.9 mm, vias 0 -> 2
- net row3: track 0.00 -> 260.9 mm, vias 0 -> 2
- net col14: track 0.00 -> 95.2 mm
- net col1: track 0.00 -> 94.6 mm
- net col2: track 0.00 -> 92.8 mm
- net col13: track 0.00 -> 90.3 mm
- net col9: track 0.00 -> 88.7 mm
- net col5: track 0.00 -> 87.9 mm
- net col10: track 0.00 -> 87.5 mm
- net col11: track 0.00 -> 86.4 mm
- net col0: track 0.00 -> 85.6 mm
- net col12: track 0.00 -> 85.1 mm
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Other:
- board outline added: 304.8 x 102.1 mm

Commit message: Final Design
Finished the D-/D+ (Differential Pair) on the USB, finished all silkscreens, and finalized all cooper traces.
Parts:
- SW10, SW11, SW12, SW13, SW14, SW16, SW18, SW19, SW2, SW20, SW21, SW22, SW23, SW24, SW25, SW26, SW27, SW28, SW29, SW3, SW31, SW33, SW34, SW35, SW36, SW37, SW38, SW39, SW4, SW40, SW41, SW42, SW43, SW46, SW48, SW49, SW5, SW50, SW51, SW52, SW53, SW54, SW55, SW56, SW57, SW6, SW60, SW61, SW7, SW72, SW73, SW74, SW75, SW76, SW77, SW8, SW9: footprint Button_Switch_Keyboard:SW_Cherry_MX_1.00u_PCB -> Custom_Switches:SW_Cherry_MX_1.00u_PCB
- SW15: footprint Button_Switch_Keyboard:SW_Cherry_MX_2.00u_PCB -> Custom_Switches:SW_Cherry_MX_2.00u_PCB
- SW17, SW30: footprint Button_Switch_Keyboard:SW_Cherry_MX_1.50u_PCB -> Custom_Switches:SW_Cherry_MX_1.50u_PCB
- SW32, SW59: footprint Button_Switch_Keyboard:SW_Cherry_MX_1.75u_PCB -> Custom_Switches:SW_Cherry_MX_1.75u_PCB
- SW45, SW47: footprint Button_Switch_Keyboard:SW_Cherry_MX_2.25u_PCB -> Custom_Switches:SW_Cherry_MX_2.25u_PCB
- SW62, SW63, SW64: footprint Button_Switch_Keyboard:SW_Cherry_MX_1.25u_PCB -> Custom_Switches:SW_Cherry_MX_1.25u_PCB
- moved R2 11.9 mm to (232.2, 120.0), turned to 0 degrees
- moved C3 6.63 mm to (226.5, 115.1), turned to 0 degrees
- moved SW1 6.39 mm to (238.8, 118.1), turned to 0 degrees
- moved C4 5.13 mm to (222.8, 111.2), turned to 0 degrees
- moved C2 4.35 mm to (226.5, 118.3), turned to 0 degrees
- moved Y1 3.25 mm to (221.8, 116.7), turned to 90 degrees
- moved J1 2.63 mm to (243.3, 110.3), turned to 0 degrees
- moved R3 2.56 mm to (208.7, 103.0)
- moved R4 2.55 mm to (206.4, 103.0)
- moved C7 1.89 mm to (215.4, 123.8)
- moved C5 1.41 mm to (200.5, 111.4), turned to 90 degrees
- moved USB1 1.02 mm to (208.3, 27.0)
- moved C6 0.69 mm to (201.1, 120.1)
- moved R5 0.62 mm to (210.9, 39.5)
- moved R1 0.33 mm to (203.6, 123.6)
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Connections:
- U1 pad 1: row0 -> row3
- U1 pad 36: col6 -> row4
- U1 pad 38: row1 -> col6
- U1 pad 39: row4 -> row0
- U1 pad 40: row3 -> row1
Routing:
- net GND: track 0.00 -> 255.7 mm, vias 0 -> 9
- net row0: track 285.2 -> 503.2 mm
- net row1: track 275.9 -> 484.2 mm
- net +5V: track 0.00 -> 204.2 mm, vias 0 -> 7
- net row2: track 267.9 -> 462.8 mm
- net col0: track 85.6 -> 242.8 mm, vias 0 -> 1
- net col14: track 95.2 -> 244.8 mm, vias 0 -> 1
- net col1: track 94.6 -> 226.2 mm, vias 0 -> 1
- net col13: track 90.3 -> 219.6 mm, vias 0 -> 1
- net col12: track 85.1 -> 193.7 mm, vias 0 -> 1
- net col2: track 92.8 -> 199.0 mm, vias 0 -> 1
- net col3: track 67.5 -> 162.5 mm, vias 0 -> 1
- net col11: track 86.4 -> 168.4 mm, vias 0 -> 1
- net col4: track 67.3 -> 141.8 mm, vias 0 -> 1
- net col8: track 67.3 -> 134.1 mm, vias 0 -> 1
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- added copper zone on B.Cu, net GND
- added copper zone on F.Cu, net GND
Other:
- board size 304.8 x 102.1 mm -> 304.8 x 102.9 mm
