File: matrix.kicad_sch (KiCad schematic)
At the start: 134 parts, among them SW10 8, SW11 9, SW12 0, SW13 -_, SW14 =+, SW15 BSPC, SW16 PGUP, SW17 Tab, SW18 Q, SW19 W, SW2 GRV, SW20 E, SW21 R, SW22 T, SW23 Y, SW24 U, SW25 I, SW26 O, SW27 P, SW28 [{, SW29 ]}, SW3 1, SW30 \|, SW31 PGDN, SW32 CAPS, SW33 A, SW34 S, SW35 D, SW36 F, SW37 G, SW38 H, SW39 J, SW4 2, SW40 K, SW41 L, SW42 ;:, SW43 '", SW45 ENTER, SW46 DEL, SW47 LSHIFT, SW48 Z, SW49 X, SW5 3, SW50 C, SW51 V, SW52 B, SW53 N, SW54 M, SW55 ,<, SW56 .>, SW57 /?, SW59 RSHIFT, SW6 4, SW60 UP, SW61 END, SW62 LCTL, SW63 WIN, SW64 LALT, SW68 SPC, SW7 5, SW72 RALT, SW73 FN, SW74 LEFT, SW75 DOWN, SW76 RIGHT, SW8 6, SW9 7

Commit message: Final Design
Finished the D-/D+ (Differential Pair) on the USB, finished all silkscreens, and finalized all cooper traces.
Parts:
- added D76: D, Diode_SMD:D_SOD-123, symbol Device:D
- added SW77: RALT, Button_Switch_Keyboard:SW_Cherry_MX_1.00u_PCB, symbol Switch:SW_Push
- SW72: value RALT -> FN
- SW73: value FN -> RCTL
Connections:
- net col5: now also SW68.2
- net col6: no longer SW68.2
- net col9: now also SW77.2
- net row4: now also D76.1 (K)
- new net: D76.2 (A), SW77.1
Other:
- moved on the sheet: D67, SW68
