File: Hardware/KeyboardRev1.kicad_sch (KiCad schematic)
At the start: 21 parts, among them J1 ISP, SW1 RESET, U1 MCU, U2 PRTR5V0U2X, Y1 16MHz

Commit message: Updated File organization
Other:
- note added: "16Mhz Crystal & Decoupling Capacitors for MCU"
- note added: "ATmega16U4"
- note added: "Auxiliary"
- note added: "HRO-TYPE-C-31-M-12"
- note added: "ISP & SW_PUSH"
- note added: "MCU"
- note added: "Reset Button"
- note added: "USB-C"
- company: (none) -> Andrew Wu
- title: (none) -> ATmega32U4 65% Keyboard PCB
- moved on the sheet: C1, C2, C3, C4, C5, C6, C7, C8, F1, J1, R1, R2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
