File: Hardware/matrix.kicad_sch (KiCad schematic)
At the start: 136 parts, among them SW10 8, SW11 9, SW12 0, SW13 -_, SW14 =+, SW15 BSPC, SW16 PGUP, SW17 Tab, SW18 Q, SW19 W, SW2 GRV, SW20 E, SW21 R, SW22 T, SW23 Y, SW24 U, SW25 I, SW26 O, SW27 P, SW28 [{, SW29 ]}, SW3 1, SW30 \|, SW31 PGDN, SW32 CAPS, SW33 A, SW34 S, SW35 D, SW36 F, SW37 G, SW38 H, SW39 J, SW4 2, SW40 K, SW41 L, SW42 ;:, SW43 '", SW45 ENTER, SW46 DEL, SW47 LSHIFT, SW48 Z, SW49 X, SW5 3, SW50 C, SW51 V, SW52 B, SW53 N, SW54 M, SW55 ,<, SW56 .>, SW57 /?, SW59 RSHIFT, SW6 4, SW60 UP, SW61 END, SW62 LCTL, SW63 WIN, SW64 LALT, SW68 SPC, SW7 5, SW72 FN, SW73 RCTL, SW74 LEFT, SW75 DOWN, SW76 RIGHT, SW77 RALT, SW8 6, SW9 7

Commit message: Updated File organization
Other:
- note added: "Diode & Switch Matrix"
- company: (none) -> Andrew Wu
- title: (none) -> Diode & Switch Matrix
- moved on the sheet: D1, D10, D11, D12, D13, D14, D15, D16, D17, D18, D19, D2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
